File: PCB/marine_tracker/marine_tracker.kicad_sch (KiCad schematic)
At the start: 34 parts, among them J1 Screw_Terminal_01x02, J2 Conn_ARM_JTAG_SWD_10, J4 BM04B-GHS-TBT, J5 molex_533981071, SW1 SW_Push, U1 STM32U575RGT6, U2 SHT40, U4 MIC5504-3.3YM5, U5 SAM-M10Q, U6 25CSM04T-I/SN, Y1 32kHz768, Y3 16MHz

Commit message: Component Placement + export Step file PCB
Connections:
- net GND: now also Y3.2
Changed lines of the file:
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@@
 		(pin "4"
+		)
+		(pin "2"
 		)
 		(instances

Commit message: routage + change GNSS module + add decoupling capacitor + change 0200/0400 package to 0600 package
Parts:
- removed U5: SAM-M10Q, Beuns_PCBFootprint:XCVR_SAM-M10Q-00B, symbol BeunsLibrary:SAM-M10Q
- added C18: 10u, Capacitor_SMD:C_0805_2012Metric, symbol Device:C
- added C19: 1u, Capacitor_SMD:C_0603_1608Metric, symbol Device:C
- added C20, C21, C23, C25: 100n, Capacitor_SMD:C_0603_1608Metric, symbol Device:C
- added C22, C24: 1n, Capacitor_SMD:C_0603_1608Metric, symbol Device:C
- added D1, D2, D3: LED, LED_SMD:LED_0603_1608Metric, symbol Device:LED
- added J3: USB_C_Receptacle_USB2.0_16P, Connector_USB:USB_C_Receptacle_GCT_USB4105-xx-A_16P_TopMnt_Horizontal, symbol Connector:USB_C_Receptacle_USB2.0_16P
- added J6: Conn_Coaxial, Connector_Coaxial:SMA_Amphenol_132289_EdgeMount, symbol Connector:Conn_Coaxial
- added R10, R8, R9: 470, Resistor_SMD:R_0402_1005Metric, symbol Device:R
- added R11: 10k, Resistor_SMD:R_0402_1005Metric, symbol Device:R
- added R12: 1k, Resistor_SMD:R_0402_1005Metric, symbol Device:R
- added R4, R7: 5k1, Resistor_SMD:R_0402_1005Metric, symbol Device:R
- added U3: MCP73833-xxx-UN, Package_SO:MSOP-10_3x3mm_P0.5mm, symbol Battery_Management:MCP73833-xxx-UN
- added U7: MAX-M10S, RF_GPS:ublox_MAX, symbol RF_GPS:MAX-M10S
- C10, C17, C3, C4, C5, C8, C9: footprint Capacitor_SMD:C_01005_0402Metric -> Capacitor_SMD:C_0603_1608Metric; JLCPCB Part Number C77008 -> (none); Manufacturer Murata Electronics -> (none); Manufacturer Part Number GRM155R61E104KA87D -> (none)
- C11, C12: footprint Capacitor_SMD:C_0402_1005Metric -> Capacitor_SMD:C_0603_1608Metric; JLCPCB Part Number C76945 -> (none); Manufacturer Murata Electronics -> (none); Manufacturer Part Number GRM1555C1H100GA01D -> (none)
- C13, C14: footprint Capacitor_SMD:C_0402_1005Metric -> Capacitor_SMD:C_0603_1608Metric; JLCPCB Part Number C76959 -> (none); Manufacturer Murata Electronics -> (none); Manufacturer Part Number GRM1555C1H200JA01D -> (none)
- C15, C16, C6: footprint Capacitor_SMD:C_0201_0603Metric -> Capacitor_SMD:C_0603_1608Metric
- C7: footprint Capacitor_SMD:C_0201_0603Metric -> Capacitor_SMD:C_0603_1608Metric; JLCPCB Part Number C77046 -> (none); Manufacturer Murata Electronics -> (none); Manufacturer Part Number GRM188R61E105KA12D -> (none)
- U6: footprint Package_SO:SOIC-8-1EP_3.9x4.9mm_P1.27mm_EP2.29x3mm -> Package_SO:JEITA_SOIC-8_3.9x4.9mm_P1.27mm
Connections:
- net +3V3: now also C20.1, C21.1, C22.1, C25.1, U7.7 (VCC_IO), U7.8 (VCC)
- net +BATT: now also C19.1, C23.1, C24.1, U3.10 (V_{BAT}), U3.9 (V_{BAT})
- net GND: now also C18.2, C19.2, C20.2, C21.2, C22.2, C23.2, C24.2, C25.2, J3.A1 (GND), J3.A12 (GND), J3.B1 (GND), J3.B12 (GND), J3.S1 (SHIELD), J6.2 (Ext), R11.2, R12.2, R4.2, R7.2, U3.5 (V_{SS}), U7.1 (GND), U7.10 (GND), U7.12 (GND)
- net GPS_EXTINT: now also U7.5 (EXTINT)
- net GPS_N_RST: now also U7.9 (~{RESET})
- net GPS_PULSE: now also U7.4 (TIMEPULSE)
- net GPS_RXD: now also U7.3 (RXD)
- net GPS_TXD: now also U7.2 (TXD)
- net MEM_SPI1_SCK: now also U1.51 (PC10); no longer U1.15 (PA1), U6.6 (SCK)
- net MEM_SPI3_MISO: now reaches U1.52 (PC11)
- net MEM_SPI3_MISO: now also U6.2 (SO)
- net MEM_SPI3_MOSI: now reaches U1.53 (PC12)
- net MEM_SPI3_MOSI: now also U6.5 (SI)
- net GPS_LNA_EN: now reaches U1.56 (PB4)
- net GPS_LNA_EN: now also U7.13 (LNA_EN)
- net MEM_SPI1_CS renamed MEM_SPI3_CS
- net MEM_SPI1_MISO renamed USB_D-
- net USB_D-: now also J3.A7 (D-), J3.B7 (D-); no longer U6.2 (SO)
- net MEM_SPI1_MOSI renamed USB_D+
- net USB_D+: now also J3.A6 (D+), J3.B6 (D+); no longer U6.5 (SI)
- new net LED1: D1.1 (K), R8.1
- new net LED2: D2.1 (K), R9.1
- new net LED3: D3.1 (K), R10.1
- new net MEM_SPI3_SCK: U6.6 (SCK)
- new net PG: R10.2, U3.7 (~{PG})
- new net PROG: R12.1, U3.6 (PROG)
- new net RF_ANT: J6.1 (In), U7.11 (RF_IN)
- new net STAT1: R8.2, U3.3 (STAT1)
- new net STAT2: R9.2, U3.4 (STAT2)
- new net THERM: R11.1, U3.8 (THERM)
- new net USB_CC1: J3.A5 (CC1), R7.1
- new net USB_CC2: J3.B5 (CC2), R4.1
- new net VBUS: C18.1, D1.2 (A), D2.2 (A), D3.2 (A), J3.A4 (VBUS), J3.A9 (VBUS), J3.B4 (VBUS), J3.B9 (VBUS), U3.1 (V_{DD}), U3.2 (V_{DD})
- no-connect marks 31 -> 32
Other:
- note added: "COMMUNICATION"
- note added: "Connector - Satellite communication module"
- note added: "For passive antenna designs, MAX-M10S integrates an LNA followed by a SAW filter in the RF path"
- note added: "LiPo Charger"
- note added: "Lipo Battery & LDO (4.2V to 3.3V)"
- note added: "MICROCONTROLLER"
- note added: "POWER SUPPLY"
- note added: "SENSORS"
- note removed: "Connector for satellite communication module"
- note removed: "LiPo 1S (3.5V-4.2V) to 3.3V LDO"
- note removed: "Pinout - TIMEPULSE pin: Precise GNSS-synchronized clock output (typically 1PPS) - EXTINT pin: External interrupt input (used for wake-up from low-power modes). Layout requirements (Refer to SAM-M10Q Integration Manual) - Minimum ground plane size: 50mm x 50mm - Minimum clearance: 10mm from each module edges (no components or copper) - Keep supply and digital lines short on the top layer - Use sol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"
- moved on the sheet: C1, C10, C11, C12, C13, C14, C15, C16, C17, C2, C3, C4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

Commit message: PCB routage WIP
Connections:
- net MEM_SPI1_SCK is gone; now on net MEM_SPI3_SCK: U1.51 (PC10)
Changed lines of the file:
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@@
 	(wire
 		(pts
-			(xy 119.38 123.698) (xy 122.682 123.698)
+			(xy 119.38 123.698) (xy 141.986 123.698)
 		)
 		(stroke
@@
 	(wire
 		(pts
-			(xy 53.34 244.856) (xy 55.118 244.856)
+			(xy 53.34 244.856) (xy 62.738 244.856)
 		)
 		(stroke
@@
 	(wire
 		(pts
-			(xy 53.594 249.936) (xy 55.118 249.936)
+			(xy 53.594 249.936) (xy 62.738 249.936)
 		)
 		(stroke
@@
 	(wire
 		(pts
-			(xy 119.38 121.158) (xy 122.682 121.158)
+			(xy 119.38 121.158) (xy 141.986 121.158)
 		)
 		(stroke
@@
 		)
 	)
+	(label "USB_D+"
+		(at 141.986 123.698 180)
+		(effects
+			(font
+				(size 1.27 1.27)
+			)
+			(justify right bottom)
+		)
+	)
 	(label "HSE_IN"
 		(at 70.612 98.298 0)
@@
 		)
 	)
+	(label "USB_D-"
+		(at 141.986 121.158 180)
+		(effects
+			(font
+				(size 1.27 1.27)
+			)
+			(justify right bottom)
+		)
+	)
 	(label "LED3"
 		(at 97.79 252.476 0)
@@
 		)
 	)
+	(label "USB_D-"
+		(at 62.738 244.856 180)
+		(effects
+			(font
+				(size 1.27 1.27)
+			)
+			(justify right bottom)
+		)
+	)
 	(label "VCAP"
 		(at 77.47 156.718 0)
@@
 		)
 	)
+	(label "USB_D+"
+		(at 62.738 249.936 180)
+		(effects
+			(font
+				(size 1.27 1.27)
+			)
+			(justify right bottom)
+		)
+	)
 	(label "LED2"
 		(at 97.79 249.936 0)
@@
 		)
 	)
-	(global_label "USB_D-"
-		(shape input)
-		(at 55.118 244.856 0)
-		(fields_autoplaced yes)
-		(effects
-			(font
-				(size 1.143 1.143)
-				(thickness 0.2286)
-				(bold yes)
-			)
-			(justify left)
-		)
-		(property "Intersheetrefs" "${INTERSHEET_REFS}"
-			(at 65.091 244.856 0)
-			(effects
-				(font
-					(size 1.27 1.27)
-				)
-				(justify left)
-				(hide yes)
-			)
-		)
-	)
 	(global_label "PRES_I2C2_SCL"
 		(shape input)
@@
 		)
 	)
-	(global_label "MEM_SPI1_SCK"
+	(global_label "MEM_SPI3_SCK"
 		(shape input)
 		(at 81.026 138.938 180)
@@
 		)
 	)
-	(global_label "USB_D+"
-		(shape input)
-		(at 55.118 249.936 0)
-		(fields_autoplaced yes)
-		(effects
-			(font
-				(size 1.143 1.143)
-				(thickness 0.2286)
-				(bold yes)
-			)
-			(justify left)
-		)
-		(property "Intersheetrefs" "${INTERSHEET_REFS}"
-			(at 65.091 249.936 0)
-			(effects
-				(font
-					(size 1.27 1.27)
-				)
-				(justify left)
-				(hide yes)
-			)
-		)
-	)
 	(global_label "SAT_RXD"
 		(shape input)
@@
 		)
 	)
-	(global_label "USB_D-"
-		(shape input)
-		(at 122.682 121.158 0)
-		(fields_autoplaced yes)
-		(effects
-			(font
-				(size 1.143 1.143)
-				(thickness 0.254)
-				(bold yes)
-			)
-			(justify left)
-		)
-		(property "Intersheetrefs" "${INTERSHEET_REFS}"
-			(at 132.782 121.158 0)
-			(effects
-				(font
-					(size 1.27 1.27)
-				)
-				(justify left)
-				(hide yes)
-			)
-		)
-	)
 	(global_label "SAT_RTS"
 		(shape input)
@@
 				(hide yes)
 			)
-		)
-	)
-	(global_label "USB_D+"
-		(shape input)
-		(at 122.682 123.698 0)
-		(fields_autoplaced yes)
-		(effects
-			(font
-				(size 1.143 1.143)
-				(thickness 0.2286)
-				(bold yes)
-			)
-			(justify left)
-		)
-		(property "Intersheetrefs" "${INTERSHEET_REFS}"
-			(at 132.655 123.698 0)
-			(effects
-				(font
-					(size 1.27 1.27)
-				)
-				(justify left)
-				(hide yes)
-			)

Commit message: add new connector for Satellite module + new LDO regulator with an maximum current higher
Parts:
- removed C16: 1u, Capacitor_SMD:C_0603_1608Metric, symbol Device:C
- removed C23: 100n, Capacitor_SMD:C_0603_1608Metric, symbol Device:C
- removed C24: 1n, Capacitor_SMD:C_0603_1608Metric, symbol Device:C
- removed J5: molex_533981071, Beuns_PCBFootprint:CONN10_533981071_MOL, symbol BeunsLibrary:molex_533981071
- removed U4: MIC5504-3.3YM5, Package_TO_SOT_SMD:SOT-23-5, symbol Regulator_Linear:MIC5504-3.3YM5
- added C26: 4u7, Capacitor_SMD:C_0603_1608Metric, symbol Device:C
- added C28: 1u, Capacitor_SMD:C_0603_1608Metric, symbol Device:C
- added J5: Conn_01x08_Pin, Connector_PinHeader_2.54mm:PinHeader_1x08_P2.54mm_Vertical, symbol Connector:Conn_01x08_Pin
- added U5: MCP1726-3302E/SN, Beuns_PCBFootprint:SOIC8-N_MC_MCH, symbol BeunsLibrary:MCP1726-3302E_SN
- C15: value 1u -> 100n; JLCPCB Part Number C77046 -> (none); Manufacturer Murata Electronics -> (none); Manufacturer Part Number GRM188R61E105KA12D -> (none)
Connections:
- net +3V3: now also C15.1, C28.1, J5.1 (Pin_1), J5.8 (Pin_8), U5.7 (VOUT), U5.8 (VOUT)
- net +BATT: now also C26.1, U5.1 (VIN), U5.2 (VIN), U5.3 (*SHDN); no longer C15.1
- net GND: now also C26.2, C28.2, J5.4 (Pin_4), J5.5 (Pin_5), U5.4 (GND)
- net SAT_RXD: now also J5.2 (Pin_2)
- net SAT_TXD: now also J5.3 (Pin_3)
- net SAT_CTS renamed SAT_VPA_EN
- net SAT_VPA_EN: now also J5.6 (Pin_6)
- net SAT_NetAv: no longer names the net of U1.22 (PA6)
- net SAT_OnOff: no longer names the net of U1.41 (PA8)
- net SAT_RI: no longer names the net of U1.23 (PA7)
- net SAT_RTS renamed SAT_VPA_SEL
- net SAT_VPA_SEL: now also J5.7 (Pin_7)
- no-connect marks 32 -> 36
Other:
- note added: "Input range : 2.3V to 6V Output : 3.3V Output current : 1A"
- note removed: "Input range : 2.5V to 5.5V Output : 3.3V Output current : 300mA"
- moved on the sheet: J1

Commit message: change to UFL connector + add stiching via
Parts:
- added C16: 100n, Capacitor_SMD:C_0603_1608Metric, symbol Device:C
- J6: footprint Connector_Coaxial:SMA_Amphenol_132289_EdgeMount -> Beuns_PCBFootprint:CONN_UFL_RSP-122811-01_SAI; Digikey Part Number ACX1426-ND -> (none); Manufacturer Amphenol RF -> (none); Manufacturer Part Number 132289 -> (none)
Connections:
- net +3V3: now also C16.1
- net GND: now also J6.3 (Ext2), C16.2

Commit message: add reference to symbols
Parts:
- removed SW1: SW_Push, Button_Switch_SMD:SW_Tactile_SPST_NO_Straight_CK_PTS636Sx25SMTRLFS, symbol Switch:SW_Push
- added SW2: SW_Push, Beuns_PCBFootprint:SW4_PTS815 SJM 250 SMTR LFS_CNK_btnPoussoir, symbol BeunsLibrary:PTS815_SJM_250_SMTR_LFS
- J2: Digikey Part Number (none) -> 609-3712-ND; JLCPCB Part Number C239059 -> (none)
- J3: Digikey Part Number (none) -> 2073-USB4215-03-ATR-ND; JLCPCB Part Number C52750322 -> (none); Manufacturer SHETIME -> GCT; Manufacturer Part Number TPS10-N1F1-2016-A -> USB4215-03-A
- J5: Digikey Part Number (none) -> 732-5321-ND; MANUFACTURER_PART_NUMBER (none) -> 61300811121; Manufacturer (none) -> Würth Elektronik
- J6: Digikey Part Number (none) -> 612-RSP-122811-01TR-ND; Manufacturer (none) -> Samtec Inc.; Manufacturer Part Number (none) -> RSP-122811-01
- U1: Digikey Part Number (none) -> 497-STM32U575RGT6-ND; JLCPCB Part Number C5270980 -> (none)
- U2: Digikey Part Number (none) -> 1649-SHT40-AD1B-R3TR-ND; JLCPCB Part Number C2848306 -> (none); Manufacturer Sensirion -> Sensirion AG
- U3: Digikey Part Number (none) -> MCP73833T-FCI/UNTR-ND; JLCPCB Part Number C627671 -> (none); Manufacturer Microchip Tech -> Microchip Technology
- U5: Digikey Part Number (none) -> MCP1726-3302E/SN-ND; Manufacturer (none) -> Microchip Technology; Manufacturer Part Number (none) -> MCP1726-3302E/SN
- U6: Digikey Part Number (none) -> 150-25CSM04T-I/SNTR-ND; JLCPCB Part Number C1513065 -> (none)
- U7: Digikey Part Number (none) -> 672-MAX-M10S-00BTR-ND; Manufacturer (none) -> u-blox; Manufacturer Part Number (none) -> MAX-M10S-00B
- Y1: Digikey Part Number (none) -> SER4071TR-ND; JLCPCB Part Number C6554955 -> (none)
- Y3: Digikey Part Number (none) -> SER4396TR-ND; JLCPCB Part Number C16171 -> (none)
Connections:
- net +3V3: now also SW2.3, SW2.4
- net BOOT0: now also SW2.1, SW2.2

Commit message: correction PCB
Parts:
- added C23: 1n, Capacitor_SMD:C_0603_1608Metric, symbol Device:C
- added C24, C27, C29, C30: 10u, Capacitor_SMD:C_0805_2012Metric, symbol Device:C
- R12: value 1k -> 2k; JLCPCB Part Number C60488 -> (none)
- U3: footprint Package_SO:MSOP-10_3x3mm_P0.5mm -> Beuns_PCBFootprint:lipo_charger; Digikey Part Number MCP73833T-FCI/UNTR-ND -> MCP73833T-FCI/MFTR-ND; Manufacturer Part Number MCP73833T-FCI/UN -> MCP73833T-FCI/MF
- U5: footprint Beuns_PCBFootprint:SOIC8-N_MC_MCH -> Beuns_PCBFootprint:LDO_1A; Digikey Part Number MCP1726-3302E/SN-ND -> MCP1726-3302E/MF-ND; Manufacturer Part Number MCP1726-3302E/SN -> MCP1726-3302E/MF
Connections:
- net +3V3: now also C24.1, C27.1, C29.1, C30.1
- net GND: now also U3.11 (EP), U5.9 (EP), C23.2, C24.2, C27.2, C29.2, C30.2
- net at U5.6 (CDELAY): now also C23.1
- no-connect marks 36 -> 35
Other:
- moved on the sheet: C15, C16, C20, C28, J4, J5

Commit message: final review + add part number
Parts:
- C1: Digikey Part Number (none) -> 311-1907-2-ND; JLCPCB Part Number C77077 -> (none); Manufacturer Murata Electronics -> YAGEO; Manufacturer Part Number GRM21BR61E475KA12L -> CC0805ZKY5V7BB475
- C10, C15, C16, C17, C20, C21, C25, C3, C4, C5, C8, C9: Digikey Part Number (none) -> 311-1088-2-ND; Manufacturer (none) -> YAGEO; Manufacturer Part Number (none) -> CC0603KRX7R7BB104
- C11, C12: Digikey Part Number (none) -> 311-1058-2-ND; Manufacturer (none) -> YAGEO; Manufacturer Part Number (none) -> CC0603JRNPO9BN100
- C13, C14: Digikey Part Number (none) -> 311-1754-2-ND; Manufacturer (none) -> YAGEO; Manufacturer Part Number (none) -> CC0603JRNPO0BN200
- C18, C2: Digikey Part Number (none) -> 311-3502-2-ND; JLCPCB Part Number C77073 -> (none); Manufacturer Murata Electronics -> YAGEO; Manufacturer Part Number GRM21BR61A106KE19L -> CC0805KRX5R7BB106
- C19, C6: Digikey Part Number (none) -> 311-1446-2-ND; JLCPCB Part Number C77046 -> (none); Manufacturer Murata Electronics -> YAGEO; Manufacturer Part Number GRM188R61E105KA12D -> CC0603KRX7R7BB105
- C22, C23: Digikey Part Number (none) -> 13-CC0603JPNPO9BN102TR-ND; Manufacturer (none) -> YAGEO; Manufacturer Part Number (none) -> CC0603JPNPO9BN102
- C24, C27, C29, C30: Digikey Part Number (none) -> 311-3502-2-ND; Manufacturer (none) -> YAGEO; Manufacturer Part Number (none) -> CC0805KRX5R7BB106
- C26: Digikey Part Number (none) -> 311-1785-2-ND; Manufacturer (none) -> YAGEO; Manufacturer Part Number (none) -> CC0603KRX5R7BB475
- C28, C7: Digikey Part Number (none) -> 311-1446-2-ND; Manufacturer (none) -> YAGEO; Manufacturer Part Number (none) -> CC0603KRX7R7BB105
- D1, D2, D3: Digikey Part Number (none) -> SML-D12U1WT86TR-ND; JLCPCB Part Number C2286 -> (none); Manufacturer Hubei KENTO Elec -> Rohm Semiconductor; Manufacturer Part Number KT-0603R -> SML-D12U1WT86
- J1: Digikey Part Number (none) -> 732-10955-ND; JLCPCB Part Number C3703 -> (none); Manufacturer Ningbo Kangnex Elec -> Würth Elektronik; Manufacturer Part Number WJ127-5.0-02P-14-00A -> 691137710002
- J4: Digikey Part Number 455-BM04B-GHS-TBTDKR-ND -> 455-BM04B-GHS-TBTTR-ND
- J5: MANUFACTURER_PART_NUMBER 61300811121 -> (none); Manufacturer Part Number (none) -> 61300811121
- R1, R11, R2, R3, R5, R6: Digikey Part Number (none) -> 311-10.0KLRTR-ND; JLCPCB Part Number C695179 -> (none); Manufacturer Part Number YC122-JR-0710KL -> RC0402FR-0710KL
- R10, R8, R9: Digikey Part Number (none) -> 311-470LRTR-ND; JLCPCB Part Number C114877 -> (none)
- R12: Digikey Part Number (none) -> 311-2KLRTR-ND
- R4, R7: Digikey Part Number (none) -> 311-5.10KLRTR-ND; JLCPCB Part Number C105872 -> (none)
