File: PCB/marine_tracker/marine_tracker.kicad_sch (KiCad schematic)
At the start: 60 parts, among them J1 Screw_Terminal_01x02, J2 Conn_ARM_JTAG_SWD_10, J3 USB_C_Receptacle_USB2.0_16P, J4 BM04B-GHS-TBT, J5 Conn_01x08_Pin, J6 Conn_Coaxial, SW2 SW_Push, U1 STM32U575RGT6, U2 SHT40, U3 MCP73833-xxx-UN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

Commit message: adding testpoint
Parts:
- added TP1, TP12, TP13, TP14, TP2, TP3, TP8, TP9: TestPoint, TestPoint:TestPoint_Pad_D1.0mm, symbol Connector:TestPoint
- added TP10, TP11, TP4, TP5, TP6, TP7: TestPoint, Connector_PinHeader_2.54mm:PinHeader_1x01_P2.54mm_Vertical, symbol Connector:TestPoint
Connections:
- net +3V3: now also TP1.1
- net +BATT: now also TP3.1
- net GND: now also TP2.1, TP7.1
- net GPS_PULSE: now also TP4.1
- net GPS_RXD: now also TP5.1
- net GPS_TXD: now also TP6.1
- net MEM_SPI3_MISO: now also TP14.1
- net MEM_SPI3_MOSI: now also TP13.1
- net MEM_SPI3_SCK: now also TP12.1
- net PRES_I2C2_SCL: now also TP10.1
- net PRES_I2C2_SDA: now also TP11.1
- net SHT_SCL: now also TP8.1
- net SHT_SDA: now also TP9.1
Other:
- moved on the sheet: C17, C25, R5, R6, U2, U6
